File: LDO_KiCad/LDO_Power.kicad_sch (KiCad schematic)
At the start: 7 parts, among them U1 TPS7A8101DRBR

Commit message: Standardize every resistor footprint to the required 0805 package
Assign Resistor_SMD:R_0805_2012Metric to all system resistors R1-R9
and both resistors in the reusable LDO schematic. This meets the
team's requirement that every resistor use 0805, fills the five
missing system resistor footprints, and replaces existing 0603
assignments. Document the requirement and remaining part-rating checks.

Validation: the installed KiCad 0805 footprint exists. Exported
before/after system netlists confirm all nine resistor footprints are
0805 and every component value and electrical net connection is
unchanged. Resistance tolerances are preserved. git diff --check passed.

Purchasing parts must still match the specified resistance/tolerance
and provide suitable power and working-voltage ratings.
Parts:
- R1, R2: footprint Resistor_SMD:R_0603_1608Metric -> Resistor_SMD:R_0805_2012Metric
Changed lines of the file:
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@@
 			)
 		)
-		(property "Footprint" "Resistor_SMD:R_0603_1608Metric"
+		(property "Footprint" "Resistor_SMD:R_0805_2012Metric"
 			(at 165.1 116.84 0)
 			(hide yes)
@@
 			)
 		)
-		(property "Footprint" "Resistor_SMD:R_0603_1608Metric"
+		(property "Footprint" "Resistor_SMD:R_0805_2012Metric"
 			(at 165.1 88.9 0)
 			(hide yes)

Commit message: Select datasheet-backed power capacitors and inductor footprints
Assign the ten missing buck capacitor footprints and L1, with actual
manufacturer part numbers, ratings and source links. Select 1210
Murata capacitors for the TPSM63606 input/output banks, 0603 ceramics
for bypass/bootstrap/feedforward roles, and a 50 V TDK 2220 part for
the existing 22 uF TPS54202 input capacitor. Keep all capacitances.
Complete LDO noise/bypass capacitor part numbers and replace the input
capacitor ordering number with a matching 1 uF 16 V 0603 Murata part;
keep the reusable LDO example consistent.

Change L1 from 10 uH to 15 uH and select Coilcraft XAL6060-153MEC.
At 2 A output, 28 V input, 390 kHz and -20% inductance tolerance,
estimated peak current is 2.439 A rather than 2.658 A for 10 uH.
The selected part has 5.8 A typical saturation current, 4.5 A thermal
reference current at 20 C rise, and 43.75 milliohm maximum DCR.
Its installed footprint matches Coilcraft's 1.43 x 5.50 mm pads on
4.04 mm centers. Normal battery range supplied by the user is
10.8-14.6 V; no bounded motor-transient voltage is assumed.

References:
TI TPSM63606 SLVSGB4B Rev. B, Tables 8-1/8-2/8-3, pp. 16-17,
and section 9.2.1.2.5, p. 24:
https://www.ti.com/lit/ds/symlink/tpsm63606.pdf
TI TPS54202 SLVSD26C Rev. C, section 7.2.3.5 and Table 7-2, pp. 15-17:
https://www.ti.com/lit/gpn/tps54202
Coilcraft XAL60xx Document 887 (02/25/26), pp. 1 and 4:
https://www.coilcraft.com/getmedia/ea51f14b-7f32-4dc6-8dfe-d4b70549040f/xal60xx.pdf
TDK C14 specifications and recommended land-pattern ranges:
https://product.tdk.com/en/search/capacitor/ceramic/mlcc/info?part_no=C5750X7R1H226M250KB

Provide a project-local C14 footprint using TDK's land-pattern ranges
(4.2 mm inner gap, 1.3 mm pad width, 5.0 mm pad height) instead of
assuming the generic 2220 footprint matches. Document all purchasing
candidates and sources in docs/passive-selection-review.md and JSON.

Validation: KiCad export succeeds; before/after component-pin n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
Parts:
- C1: MPN EMK107B7105KA-T -> GRM188R71C105KA12D; Manufacturer Taiyo Yuden -> Murata
- C3, C4: MPN TBD -> GRM188R71C474KA88D; Manufacturer (none) -> Murata
Changed lines of the file:
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@@
 		(property "Datasheet" ""
 			(at 165.1 116.84 0)
+			(hide yes)
 			(show_name no)
 			(do_not_autoplace no)
@@
 			)
 		)
-		(property "Datasheet" ""
+		(property "Datasheet" "https://search.murata.co.jp/Ceramy/image/img/A01X/G101/ENG/GRM188R71C474KA88-01A.pdf"
 			(at 96.52 116.84 0)
+			(hide yes)
 			(show_name no)
 			(do_not_autoplace no)
@@
 			)
 		)
-		(property "MPN" "TBD"
+		(property "MPN" "GRM188R71C474KA88D"
 			(at 96.52 116.84 0)
 			(hide yes)
@@
 				)
 			)
+		)
+		(property "Manufacturer" "Murata"
+			(at 96.52 116.84 0)
+			(hide yes)
+			(effects (font (size 1.27 1.27)))
 		)
 	)
@@
 		(property "Datasheet" ""
 			(at 210.82 106.68 0)
+			(hide yes)
 			(show_name no)
 			(do_not_autoplace no)
@@
 		(property "Datasheet" ""
 			(at 165.1 88.9 0)
+			(hide yes)
 			(show_name no)
 			(do_not_autoplace no)
@@
 			)
 		)
-		(property "Datasheet" ""
+		(property "Datasheet" "https://search.murata.co.jp/Ceramy/image/img/A01X/G101/ENG/GRM188R71C105KA12-01.pdf"
 			(at 76.2 101.6 0)
+			(hide yes)
 			(show_name no)
 			(do_not_autoplace no)
@@
 			)
 		)
-		(property "MPN" "EMK107B7105KA-T"
+		(property "MPN" "GRM188R71C105KA12D"
 			(at 76.2 101.6 0)
 			(hide yes)
@@
 			)
 		)
-		(property "Manufacturer" "Taiyo Yuden"
+		(property "Manufacturer" "Murata"
 			(at 76.2 104.14 0)
 			(hide yes)
@@
 			)
 		)
-		(property "Datasheet" ""
+		(property "Datasheet" "https://search.murata.co.jp/Ceramy/image/img/A01X/G101/ENG/GRM188R71C474KA88-01A.pdf"
 			(at 190.5 88.9 0)
+			(hide yes)
 			(show_name no)
 			(do_not_autoplace no)
@@
 			)
 		)
-		(property "MPN" "TBD"
+		(property "MPN" "GRM188R71C474KA88D"
 			(at 190.5 88.9 0)
 			(hide yes)
@@
 			)
 		)
+		(property "Manufacturer" "Murata"
+			(at 190.5 88.9 0)
+			(hide yes)
+			(effects (font (size 1.27 1.27)))
+		)
 	)
