File: Buck_5V_6A.kicad_sch (KiCad schematic)
At the start: 10 parts, among them U2 PTPSM63606RDLR

Commit message: Add motor 1 driver and encoder screw terminals
Label the STM32 pins used in the motor prototype: PA6 MOTOR1_PWM
(TIM3_CH1 to DRI0002 E1), PB0 MOTOR1_DIR (M1), PA15 ENC1_A and PB3
ENC1_B (TIM2 encoder inputs).

Add screw terminals to the right of U1:
- J6, 3-pos: MOTOR1_PWM, MOTOR1_DIR, GND for the DFRobot DRI0002
- J7, 4-pos: +5V 2A, ENC1_A, ENC1_B, GND for the 37D motor encoder
Encoder power comes from the +5V 2A buck rail ahead of the LDO.

Both use Phoenix MKDS 1,5 5.0 mm footprints (1715035, 1715048),
rated 17.5 A / 250 V for the 5 V, 2 A requirement, with datasheet,
part number and pinout stored in the symbol properties.

Also includes the sheet layout rearranged in KiCad.

Co-Authored-By: Claude Opus 5.5 <noreply@anthropic.com>
Other:
- note added: "12 V - 5 V, 6A Buck Convertor"
- note removed: "BUCK CONVERTOR 12V-5.1V, 6AMPS"
- moved on the sheet: C10, C11, C12, C7, C8, C9, R2, R4, R5, U2
