File: Buck_5V_6A.kicad_sch (KiCad schematic)
At the start: 10 parts, among them U2 PTPSM63606RDLR

Commit message: Rename power nets, add mounting holes, retitle sheet 1, clear ERC
Power nets, no commas, named by function:
- "+5V, 2A" -> +5V_SYS, "+5V, 6A PI" -> +5V_PI, "+5V, 6A AUX" -> +5V_AUX
Buck sheets renamed to Buck 5V SYS / Buck 5V PI / Buck 5V AUX. Notes,
descriptions, README and docs updated.

Mechanical and title:
- H1-H4: M3 mounting holes, 3.2 mm plated, isolated (no net), not in BOM
- Sheet 1 title: "Delivery Robot Main Board"

ERC, now 0 errors and 0 warnings (was 4 errors, 15 warnings):
- PWR_FLAGs on +12V (after F1), GND (at J2), +3.3VA (after FB2) and
  +5V_SYS (after the TPS54202's L1)
- TPSM63606 symbol pin types set (VOUT power out, FB/EN input, VIN/
  VLDOIN/GND power in, PG open collector, others passive) in both buck
  sheets and libs/TPSM63606RDLR.kicad_sym
- U1 STM32F091RCTx and Y3 Crystal_GND24 moved to a new
  libs/project_symbols.kicad_sym holding the versions this design uses
  (the current KiCad library moved their pins); libs/TPS54202DDCR made
  to match the schematic's U3
Connectivity unchanged: same 108 nets and pins.

Co-Authored-By: Claude Opus 5.5 <noreply@anthropic.com>
Parts:
- U2: Used In Sheet Buck_5V_6A: 12 V in, +5V 6A net out -> Sheet Buck_5V_6A: 12 V in, +5V_PI net out
Changed lines of the file:
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@@
 			)
 		)
-		(property "Used In" "Sheet Buck_5V_6A: 12 V in, +5V 6A net out"
+		(property "Used In" "Sheet Buck_5V_6A: 12 V in, +5V_PI net out"
 			(at 115.57 86.36 0)
 			(hide yes)

Commit message: Add input protection, AUX ports, servo interface and Pi control
Implements the 2026-10-15 design review decisions in the schematic.
ERC 0 errors, 0 warnings.

New sheets:
- Input Protection: Q1 SQJ409EP reverse-battery P-FET after F1 (D12
  12 V gate clamp, R36), D13 SMBJ16A TVS on +12V, battery sense
  R37/R38/C37 -> VBAT_SENSE on PA0. PWR_FLAG moves to +12V.
- AUX Outputs: four +5V_AUX ports J18-J21 (JST XH 2-pin: Notecard,
  LiDAR, GNSS, IMU), each through a 1.5 A PTC (F4-F7).
- Servo Interface: J17 (GND, VBAT_SERVO via F3 5 A fuse, SERVO_SIG) for
  the Hiwonder HTS-30HS through an external 11.1-12 V buck. U8
  SN74LVC1T45 translates PB10 (USART3 half-duplex) to the 5 V bus,
  PB11 sets direction; R39-R42 pull-ups/series, D14 ESD.

Root sheet:
- F1 output is now VBAT_FUSED; C36 sits on +12V after Q1. J2-F1 net
  named VBAT_IN. F1 7.5 A -> 10 A (0297010.L).
- Y3/C5/C6 fitted (were DNP).
- PA0 -> VBAT_SENSE, PA1 -> PI_3V3_SENSE, PB10 -> SERVO_TX,
  PB11 -> SERVO_DIR. Notes updated (no more F2 / XT30-only text).

Pi 5 Interface:
- J13 -> 6-pin JST XH: TXD, RXD, GND, PI_3V3, PI_RESET, PI_BOOT0.
- PI_3V3 -> D15 -> AUX_EN (U5 enable) and R44/R45 -> PA1.
- PI_RESET -> Q2 DMN63D8L -> NRST (open drain, R46 pull-down).
- PI_BOOT0 -> R47 1k -> BOOT0, for reflashing over USART2.
- R12/R13 100R -> 1k (PA2/PA3 are TTa, 5 mA injection max).
- Remove TP2 (same net as TP1 since F2 was removed).

Buck 5V AUX: U5 EN from AUX_EN (was +12V), R43 100k pull-down, C40,
J22 force-on jumper. Buck 5V SYS: C49 100 nF at U3 VIN/GND.
U2/U5 value TPSM63606RDLR; VCC design note corrected (internal 1 uF,
must stay NC).

Motor Control (now A3):
- U9/U10 74LVC2G17 encoder buffers on +3V3; encoder series R 100R ->
  1k with C43-C46 1 nF; R48-R51 4.7k pull-ups (DNP).
- F8/F9 0.2 A PTC + C47/C48 on each encoder supply (ENC1_5V, ENC2_5V).
- J7/J15 pin order 5V, GND, A, B (matches the am-3651 plug).
- R52/R53 10k pull-downs on both PWM lines (MDD20A brakes on low).
- F10/F11 PTC in series with J6/J16 p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
Parts:
- U2: value PTPSM63606RDLR -> TPSM63606RDLR; Design Notes VOUT = VREF x (1 + R4/R5) with FB divider R4 41.2k / R5 10k (VOUT = 5.12 V for the Pi 5), C10 feed-forward; RT = R2 12.1k; EN tied to VIN; RBOOT shorted to CBOOT; SW pin left NC; PG open-drain, unused; VLDOIN tied to VOUT; VCC needs 1 uF to AGND per datasheet - CHECK C9 placement (currently on VLDOIN/VOUT, VCC flagged NC) -> VOUT = VREF x (1 + R4/R5) with FB divider R4 41.2k / R5 10k (VOUT = 5.12 V for the Pi 5), C10 feed-forward; RT = R2 12.1k; EN tied to VIN; RBOOT shorted to CBOOT; SW pin left NC; PG open-drain, unused; VLDOIN tied to VOUT; VCC has an internal 1 uF and must not be loaded (SLVSGB4B pin table), so it is left NC; C9 is the VLDOIN capacitor; MPN TPSM63606RDLR (schematic symbol: PTPSM63606RDLR) -> TPSM63606RDLR
Changed lines of the file:
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@@
 			)
 		)
-		(property "Value" "PTPSM63606RDLR"
+		(property "Value" "TPSM63606RDLR"
 			(at 137.16 78.74 0)
 			(show_name no)
@@
 			)
 		)
-		(property "MPN" "TPSM63606RDLR (schematic symbol: PTPSM63606RDLR)"
+		(property "MPN" "TPSM63606RDLR"
 			(at 115.57 86.36 0)
 			(hide yes)
@@
 			)
 		)
-		(property "Design Notes" "VOUT = VREF x (1 + R4/R5) with FB divider R4 41.2k / R5 10k (VOUT = 5.12 V for the Pi 5), C10 feed-forward; RT = R2 12.1k; EN tied to VIN; RBOOT shorted to CBOOT; SW pin left NC; PG open-drain, unused; VLDOIN tied to VOUT; VCC needs 1 uF to AGND per datasheet - CHECK C9 placement (currently on VLDOIN/VOUT, VCC flagged NC)"
+		(property "Design Notes" "VOUT = VREF x (1 + R4/R5) with FB divider R4 41.2k / R5 10k (VOUT = 5.12 V for the Pi 5), C10 feed-forward; RT = R2 12.1k; EN tied to VIN; RBOOT shorted to CBOOT; SW pin left NC; PG open-drain, unused; VLDOIN tied to VOUT; VCC has an internal 1 uF and must not be loaded (SLVSGB4B pin table), so it is left NC; C9 is the VLDOIN capacitor"
 			(at 115.57 86.36 0)
 			(hide yes)
