File: delivery_robot_1.kicad_sch (KiCad schematic)
At the start: 36 parts, among them J1 SWD, J10 Port C/D breakout, J11 IMU I2C (STEMMA QT), J12 IMU INT/RST, J13 Pi 5 UART, J2 Conn_01x02, J4 BOOT0 jumper, J5 Conn_01x03_Pin, J6 DRI0002 E1/M1/GND, J7 Motor1 encoder, J8 Port A breakout, J9 Port B breakout, SW1 RESET, U1 STM32F091RCTx, Y3 8MHz

Commit message: Add fused, isolatable Pi 5 power output from the 6 A buck
Feed the off-board Raspberry Pi 5 from the +5V, 6A buck rail:
- F2: Keystone 3568 MINI holder with Littelfuse 029707.5L 7.5 A fuse,
  same verified parts as F1. Pulling the fuse isolates the Pi so the
  buck can be checked and load-tested first; fitted, it protects the
  Pi cable (6.0 A allowed at 40 C, above the Pi 5's 5 A maximum).
- J14: Phoenix MKDS 1,5/2 5.0 mm screw terminal (1715022, 17.5 A,
  26-14 AWG) for a USB-C plug pigtail: 1 = PI_5V, 2 = GND.
- TP1/TP2: Keystone 5000 test loops on the buck output and PI_5V.
Parts:
- added F2: 7.5A / 32VDC, Fuse:Fuseholder_Blade_Mini_Keystone_3568, symbol Device:Fuse
- added J14: Pi 5 power, TerminalBlock_Phoenix:TerminalBlock_Phoenix_MKDS-1,5-2_1x02_P5.00mm_Horizontal, symbol Connector:Screw_Terminal_01x02
- added TP1: +5V, 6A, TestPoint:TestPoint_Keystone_5000-5004_Miniature, symbol Connector:TestPoint
- added TP2: PI_5V, TestPoint:TestPoint_Keystone_5000-5004_Miniature, symbol Connector:TestPoint
Connections:
- net +5V, 6A: now also F2.2, TP1.1
- net GND: now also J14.2 (Pin_2)
- new net: F2.1, J14.1 (Pin_1), TP2.1
Other:
- note added: "Bring-up: F2 out, check TP1; fit F2, load-test J14; then connect the Pi. 5-6 A path"
- note added: "Pi 5 power: +5V, 6A -> F2 isolation fuse -> J14 USB-C pigtail"
- moved on the sheet: J11, J12, J13, R10, R11, R12, R13

Commit message: Switch motor 1 driver notes from DFRobot DRI0002 to Cytron MDD20A
The Cytron MDD20A (20 A, 6-30 V, 2-channel) uses the same control
interface as the DRI0002 on channel 1, so J6 wiring is unchanged:
1 = PWM1 (PA6, TIM3_CH1), 2 = DIR1 (PB0), 3 = GND. Its logic
thresholds (low <= 0.8 V, high >= 1.5 V) accept the STM32's 3.3 V
outputs; keep PWM at or below 20 kHz.

Update J6's value and description and the motor section note,
including the datasheet link and that battery VB+/VB- and motor
M1A/M1B wire directly to the driver. No connectivity changes.
Parts:
- J6: value DRI0002 E1/M1/GND -> MDD20A PWM1/DIR1/GND
Other:
- note added: "Motor 1 off-board connections (Cytron MDD20A driver + 37D encoder motor) PWM on TIM3 (PA6), encoder on TIM2 (PA15 / PB3). Encoder Vcc is +5V, 2A from the TPS54202 buck (before the LDO), not from the MCU. Driver VB+/VB- (6-30 V battery) and M1A/M1B wire directly to the MDD20A (not on this board)."
- note removed: "Motor 1 off-board connections (DFRobot DRI0002 driver + 37D encoder motor) PWM on TIM3 (PA6), encoder on TIM2 (PA15 / PB3). Encoder Vcc is +5V, 2A from the TPS54202 buck (before the LDO), not from the MCU. Driver VS/GND and Motor+/- wire directly between DRI0002 and motor (not on this board)."
Changed lines of the file:
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@@
 		)
 	)
-	(text "Motor 1 off-board connections (DFRobot DRI0002 driver + 37D encoder motor)\nPWM on TIM3 (PA6), encoder on TIM2 (PA15 / PB3).\nEncoder Vcc is +5V, 2A from the TPS54202 buck (before the LDO), not from the MCU.\nDriver VS/GND and Motor+/- wire directly between DRI0002 and motor (not on this board)."
+	(text "Motor 1 off-board connections (Cytron MDD20A driver + 37D encoder motor)\nPWM on TIM3 (PA6), encoder on TIM2 (PA15 / PB3).\nEncoder Vcc is +5V, 2A from the TPS54202 buck (before the LDO), not from the MCU.\nDriver VB+/VB- (6-30 V battery) and M1A/M1B wire directly to the MDD20A (not on this board)."
 		(exclude_from_sim no)
 		(at 181.61 26.67 0)
@@
 			)
 		)
-		(property "Value" "DRI0002 E1/M1/GND"
+		(property "Value" "MDD20A PWM1/DIR1/GND"
 			(at 218.44 46.99 0)
 			(show_name no)
@@
 			)
 		)
-		(property "Description" "Motor 1 driver control to DFRobot DRI0002: 1 = E1 speed PWM (PA6, TIM3_CH1), 2 = M1 direction (PB0), 3 = GND"
+		(property "Description" "Motor 1 driver control to Cytron MDD20A (20 A, 6-30 V, 2-channel): 1 = PWM1 speed (PA6, TIM3_CH1, max 20 kHz), 2 = DIR1 direction (PB0), 3 = GND. MDD20A logic: low <= 0.8 V, high >= 1.5 V, so 3.3 V drive is fine. Datasheet: https://cdn.robotshop.com/media/c/cyt/rb-cyt-287/pdf/cytron-20a-6v-30v-dual-dc-motor-driver-datasheet.pdf"
 			(at 214.63 46.99 0)
 			(hide yes)

Commit message: changing the connectors from the battery to the pcb
Parts:
- J2: value Conn_01x02 -> XT30PW-M; footprint (none) -> Connector_AMASS:AMASS_XT30PW-M_1x02_P2.50mm_Horizontal; MPN (none) -> XT30PW-M; Manufacturer (none) -> AMASS; MatingPart (none) -> AMASS XT30U-F on the battery harness
Connections:
- net GND: now also J2.1 (Pin_1); no longer J2.2 (Pin_2)
- net at F1.2: now also J2.2 (Pin_2); no longer J2.1 (Pin_1)
Other:
- moved on the sheet: J2
Changed lines of the file:
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@@
 	(symbol
 		(lib_id "Connector_Generic:Conn_01x02")
-		(at 35.56 161.29 0)
-		(mirror y)
+		(at 35.56 163.83 180)
 		(unit 1)
 		(body_style 1)
@@
 		(in_pos_files yes)
 		(dnp no)
-		(fields_autoplaced yes)
 		(property "Reference" "J2"
-			(at 33.02 161.2899 0)
+			(at 33.02 160.02 0)
 			(show_name no)
 			(do_not_autoplace no)
@@
 			)
 		)
-		(property "Value" "Conn_01x02"
-			(at 33.02 163.8299 0)
+		(property "Value" "XT30PW-M"
+			(at 33.02 166.37 0)
 			(show_name no)
 			(do_not_autoplace no)
@@
 			)
 		)
-		(property "Footprint" ""
+		(property "Footprint" "Connector_AMASS:AMASS_XT30PW-M_1x02_P2.50mm_Horizontal"
 			(at 35.56 161.29 0)
 			(hide yes)
@@
 			)
 		)
-		(property "Datasheet" ""
+		(property "Datasheet" "https://www.tme.eu/Document/6eb2005a51a52592b3f19e8a450c54c8/XT30PW-M.pdf"
 			(at 35.56 161.29 0)
 			(hide yes)
@@
 			)
 		)
-		(property "Description" "Generic connector, single row, 01x02, script generated (kicad-library-utils/schlib/autogen/connector/)"
+		(property "Description" "12 V battery input, AMASS XT30PW-M right-angle PCB male (15 A continuous, 30 A short-term, 500 V), keyed. Pin 2 (+ silkscreen) = battery + to F1; pin 1 (- silkscreen) = GND. Mates with an XT30U-F plug on the battery harness: DJLBERMPW 12V 50Ah LiFePO4 M8 terminals -> M8 ring lugs -> inline fuse at the battery -> 16 AWG -> XT30U-F."
 			(at 35.56 161.29 0)
 			(hide yes)
 			(show_name no)
+			(do_not_autoplace no)
+			(effects
+				(font
+					(size 1.27 1.27)
+				)
+			)
+		)
+		(property "Manufacturer" "AMASS"
+			(at 35.56 163.83 0)
+			(hide yes)
+			(show_name no)
+			(do_not_autoplace no)
+			(effects
+				(font
+					(size 1.27 1.27)
+				)
+			)
+		)
+		(property "MPN" "XT30PW-M"
+			(at 35.56 163.83 0)
+			(hide yes)
+			(show_name no)
+			(do_not_autoplace no)
+			(effects
+				(font
+					(size 1.27 1.27)
+				)
+			)
+		)
+		(property "MatingPart" "AMASS XT30U-F on the battery harness"
+			(at 35.56 163.83 0)
+			(hide yes)
+			(show_name no)
