File: Buck_5V_6A_AUX.kicad_sch (KiCad schematic)
At the start: 10 parts, among them U5 PTPSM63606RDLR

Commit message: Add +12V bulk capacitor, document XT30 polarity decision, use E96 values
Input (sheet 1, near J2):
- C36: 220 uF / 35 V low-ESR electrolytic (Panasonic EEU-FR1V221,
  8 x 11.5 mm radial) on +12V right after F1.
- Reverse polarity: no P-FET; rely on the keyed XT30. Note on sheet 1
  and in docs/power-supply.md: the housing cannot mate reversed, but a
  harness crimped backwards at the battery lugs is not caught (it would
  reverse-bias both bucks and C36 until F1 blows), so meter-check harness
  polarity before first power-up and after rework.

All resistor values are now E96:
- R4 40k -> 41.2k 1%: Pi rail 5.12 V (5.1 V target)
- R15 40k -> 40.2k 1%: AUX rail 5.02 V
- R8/R9 31.2k/10k -> 35.7k/11.5k: LDO 3.284 V (31.2k is E192)
- R3 510 -> 511, R21-R24 680 -> 681, R17/R10/R11 4.7k -> 4.75k
Regulator design notes, sheet notes and docs updated to match.
Parts:
- R15: value 40kOhms -> 40.2k / 1%
- U5: Design Notes VOUT = VREF x (1 + R15/R16) with FB divider R15 40k / R16 1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 -> VOUT = VREF x (1 + R15/R16) with FB divider R15 40.2k / R16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
Changed lines of the file:
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@@
 			)
 		)
-		(property "Value" "40kOhms"
+		(property "Value" "40.2k / 1%"
 			(at 179.07 93.98 0)
 			(show_name no)
@@
 			)
 		)
-		(property "Design Notes" "VOUT = VREF x (1 + R15/R16) with FB divider R15 40k / R16 10k, C31 feed-forward; RT = R14 12.1k; EN tied to VIN; RBOOT shorted to CBOOT; SW pin left NC; PG open-drain, unused; VLDOIN tied to VOUT; VCC needs 1 uF to AGND per datasheet - CHECK C30 placement (currently on VLDOIN/VOUT, VCC flagged NC)"
-			(at 115.57 86.36 0)
-			(hide yes)
+		(property "Design Notes" "VOUT = VREF x (1 + R15/R16) with FB divider R15 40.2k / R16 10k (VOUT = 5.02 V), C31 feed-forward; RT = R14 12.1k; EN tied to VIN; RBOOT shorted to CBOOT; SW pin left NC; PG open-drain, unused; VLDOIN tied to VOUT; VCC needs 1 uF to AGND per datasheet - CHECK C30 placement (currently on VLDOIN/VOUT, VCC flagged NC)"
+			(at 115.57 86.36 0)
+			(hide yes)
