File: Buck_5V_6A_AUX.kicad_sch (KiCad schematic)
At the start: 15 parts, among them J22 AUX force-on, U5 TPS56637RPAR

Commit message: Apply TA layout review: vias off pads, obtuse corners, buck layouts
- Move every via off its pad. The +3V3 vias at U6/U11/C34/C50 sit
  0.03-0.06 mm from the pad edge, without overlap, and are tented.
- Remove the remaining acute and right-angle track corners, including
  where tracks leave a pad, and straighten small jogs (R27 pin 2).
- U2/U5: add a second 47 uF output cap (C57, C58) to match the
  two-Cout datasheet layout, and add more PGND vias. F1 moves up 1 mm
  to make room for C57.
- U3: move C14 down 1 mm so the input cap GND pads have a via on each
  side.

DRC: 0 violations, 0 unconnected, 0 parity issues. ERC clean.
Parts:
- added C58: 47uF, Capacitor_SMD:C_1210_3225Metric, symbol Device:C
Connections:
- net GND: now also C58.2
- net VOUT_5V: now also C58.1
Changed lines of the file:
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@@
+		)
+	)
+	(symbol
+		(lib_id "Device:C")
+		(at 186.69 107.95 0)
+		(unit 1)
+		(body_style 1)
+		(exclude_from_sim no)
+		(in_bom yes)
+		(on_board yes)
+		(in_pos_files yes)
+		(dnp no)
+		(property "Reference" "C58"
+			(at 190.5 106.68 0)
+			(show_name no)
+			(do_not_autoplace no)
+			(effects (font (size 1.27 1.27)) (justify left))
+		)
+		(property "Value" "47uF"
+			(at 190.5 109.22 0)
+			(show_name no)
+			(do_not_autoplace no)
+			(effects (font (size 1.27 1.27)) (justify left))
+		)
+		(property "Footprint" "Capacitor_SMD:C_1210_3225Metric"
+			(at 186.69 113.03 0)
+			(hide yes)
+			(show_name no)
+			(do_not_autoplace no)
+			(effects (font (size 1.27 1.27)) (justify left))
+		)
+		(property "Datasheet" "https://search.murata.co.jp/Ceramy/image/img/A01X/G101/ENG/GRM32ER61C476KE15-01.pdf"
+			(at 186.69 113.03 0)
+			(hide yes)
+			(show_name no)
+			(do_not_autoplace no)
+			(effects (font (size 1.27 1.27)) (justify left))
+		)
+		(property "Description" "Unpolarized capacitor"
+			(at 186.69 113.03 0)
+			(hide yes)
+			(show_name no)
+			(do_not_autoplace no)
+			(effects (font (size 1.27 1.27)) (justify left))
+		)
+		(property "Manufacturer" "Murata"
+			(at 186.69 113.03 0)
+			(hide yes)
+			(show_name no)
+			(do_not_autoplace no)
+			(effects (font (size 1.27 1.27)) (justify left))
+		)
+		(property "MPN" "GRM32ER61C476KE15L"
+			(at 186.69 113.03 0)
+			(hide yes)
+			(show_name no)
+			(do_not_autoplace no)
+			(effects (font (size 1.27 1.27)) (justify left))
+		)
+		(property "Specification" "47uF / 16V X5R 1210 (Cout)"
+			(at 186.69 113.03 0)
+			(hide yes)
+			(show_name no)
+			(do_not_autoplace no)
+			(effects (font (size 1.27 1.27)) (justify left))
+		)
+		(pin "1")
+		(pin "2")
+		(instances
+			(project "delivery_robot_1"
+				(path "/30314d9c-15a8-4a77-8ae4-b5ba12ed5bc4/472ee453-7701-4e13-8d8d-09d254496392"
+					(reference "C58")
+					(unit 1)
+				)
+			)
 		)
 	)
 	(wire
+		(pts (xy 186.69 104.14) (xy 186.69 101.6))
+		(stroke (width 0) (type default))
+	)
+	(wire
+		(pts (xy 186.69 101.6) (xy 176.53 101.6))
+		(stroke (width 0) (type default))
+	)
+	(wire
+		(pts (xy 186.69 111.76) (xy 186.69 114.3))
+		(stroke (width 0) (type default))
+	)
+	(wire
+		(pts (xy 186.69 114.3) (xy 176.53 114.3))
+		(stroke (width 0) (type default))
+	)
+	(junction
+		(at 176.53 101.6)
+		(diameter 0)
+		(color 0 0 0 0)
+	)
+	(junction
+		(at 176.53 114.3)
+		(diameter 0)
+		(color 0 0 0 0)
+	)
+	(wire
 		(pts (xy 176.53 104.14) (xy 176.53 101.6))
