File: IMU_Interface.kicad_sch (KiCad schematic)
At the start: 6 parts, among them J11 IMU I2C (STEMMA QT), J12 IMU INT/RST

Commit message: Add +12V bulk capacitor, document XT30 polarity decision, use E96 values
Input (sheet 1, near J2):
- C36: 220 uF / 35 V low-ESR electrolytic (Panasonic EEU-FR1V221,
  8 x 11.5 mm radial) on +12V right after F1.
- Reverse polarity: no P-FET; rely on the keyed XT30. Note on sheet 1
  and in docs/power-supply.md: the housing cannot mate reversed, but a
  harness crimped backwards at the battery lugs is not caught (it would
  reverse-bias both bucks and C36 until F1 blows), so meter-check harness
  polarity before first power-up and after rework.

All resistor values are now E96:
- R4 40k -> 41.2k 1%: Pi rail 5.12 V (5.1 V target)
- R15 40k -> 40.2k 1%: AUX rail 5.02 V
- R8/R9 31.2k/10k -> 35.7k/11.5k: LDO 3.284 V (31.2k is E192)
- R3 510 -> 511, R21-R24 680 -> 681, R17/R10/R11 4.7k -> 4.75k
Regulator design notes, sheet notes and docs updated to match.
Parts:
- R10, R11: value 4.7k -> 4.75k
Changed lines of the file:
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@@
 			)
 		)
-		(property "Value" "4.7k"
+		(property "Value" "4.75k"
 			(at 82.55 105.41 0)
 			(show_name no)
@@
 			)
 		)
-		(property "Description" "Optional IMU_SCL pull-up to +3V3, DNP: the Adafruit BNO085 breakout already has pull-ups. Fit 4.7k if the breakout lacks them or the bus misbehaves over the cable."
+		(property "Description" "Optional IMU_SCL pull-up to +3V3, DNP: the Adafruit BNO085 breakout already has pull-ups. Fit 4.75k if the breakout lacks them or the bus misbehaves over the cable."
 			(at 80.01 104.14 0)
 			(hide yes)
@@
 			)
 		)
-		(property "Value" "4.7k"
+		(property "Value" "4.75k"
 			(at 62.23 105.41 0)
 			(show_name no)
@@
 			)
 		)
-		(property "Description" "Optional IMU_SDA pull-up to +3V3, DNP: the Adafruit BNO085 breakout already has pull-ups. Fit 4.7k if the breakout lacks them or the bus misbehaves over the cable."
+		(property "Description" "Optional IMU_SDA pull-up to +3V3, DNP: the Adafruit BNO085 breakout already has pull-ups. Fit 4.75k if the breakout lacks them or the bus misbehaves over the cable."
 			(at 59.69 104.14 0)
 			(hide yes)
