File: LDO_3V3.kicad_sch (KiCad schematic)
At the start: 7 parts, among them U4 TPS7A8101DRBR

Commit message: Route the board and apply the prototype PCB checklist fixes
Routing
- Route power (pours, In2 power areas, vias) and all signals; add a
  Signal net class (0.15 mm width/clearance) for low-speed nets.
- J8 expansion header is now a 2x8 near the MCU.

Checklist red flags
- Crystal Y3 moved beside U1's OSC pins with C5/C6 outboard and no
  other signals under it.
- Vias untented by default (tented only under silkscreen); 15 mil
  test vias on key signals, recorded as DRC exclusions.
- ESD: U6/U7 split into four USBLC6-2SC6 (U6, U11, U7, U12), one per
  connector, with VBUS caps C50/C51; R12/R13 moved next to J13.
- GND test loop TP3 moved to the top edge beside J5.

Improvements
- Encoder connectors J7/J15 changed to keyed JST XH S4B side-entry.
- 43 passives/LEDs/FB2 moved from 0603 to 0805 (MPNs updated).
- Fifth M3 mounting hole H5 under J8.
- +3.3VA rerouted away from the crystal; acute track angles removed.
- Datasheet links filled in; silkscreen pin labels, pin maps, team
  names and date; reference labels cleared off pads and vias.
- Custom DRC rule for the J7/J15 silkscreen edge overhang.
Parts:
- C24: footprint Capacitor_SMD:C_0603_1608Metric -> Capacitor_SMD:C_0805_2012Metric; MPN GRM188R71C105KA12D -> GRM21BR71C105KA01L
- C26, C27: footprint Capacitor_SMD:C_0603_1608Metric -> Capacitor_SMD:C_0805_2012Metric; MPN GRM188R72A103KA01D -> GRM21BR72A103KA01L
Changed lines of the file:
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@@
 			)
 		)
-		(property "Footprint" "Capacitor_SMD:C_0603_1608Metric"
+		(property "Footprint" "Capacitor_SMD:C_0805_2012Metric"
 			(at 96.52 116.84 0)
 			(hide yes)
@@
 			)
 		)
-		(property "Datasheet" ""
+		(property "Datasheet" "https://www.murata.com/en-us/products/productdetail?partno=GRM21BR72A103KA01%23"
 			(at 96.52 116.84 0)
 			(hide yes)
@@
 			)
 		)
-		(property "MPN" "GRM188R72A103KA01D"
+		(property "MPN" "GRM21BR72A103KA01L"
 			(at 96.52 116.84 0)
 			(hide yes)
@@
 			)
 		)
-		(property "Datasheet" ""
+		(property "Datasheet" "https://product.tdk.com/en/search/capacitor/ceramic/mlcc/info?part_no=C2012X7R1A106K125AC"
 			(at 210.82 106.68 0)
 			(hide yes)
@@
 			)
 		)
-		(property "Footprint" "Capacitor_SMD:C_0603_1608Metric"
+		(property "Footprint" "Capacitor_SMD:C_0805_2012Metric"
 			(at 76.2 101.6 0)
 			(hide yes)
@@
 			)
 		)
-		(property "Datasheet" "https://search.murata.co.jp/Ceramy/image/img/A01X/G101/ENG/GRM188R71C105KA12-01.pdf"
+		(property "Datasheet" "https://www.murata.com/en-us/products/productdetail?partno=GRM21BR71C105KA01%23"
 			(at 76.2 101.6 0)
 			(hide yes)
@@
 			)
 		)
-		(property "MPN" "GRM188R71C105KA12D"
+		(property "MPN" "GRM21BR71C105KA01L"
 			(at 76.2 101.6 0)
 			(hide yes)
@@
 			)
 		)
-		(property "Footprint" "Capacitor_SMD:C_0603_1608Metric"
+		(property "Footprint" "Capacitor_SMD:C_0805_2012Metric"
 			(at 190.5 88.9 0)
 			(hide yes)
@@
 			)
 		)
-		(property "Datasheet" ""
+		(property "Datasheet" "https://www.murata.com/en-us/products/productdetail?partno=GRM21BR72A103KA01%23"
 			(at 190.5 88.9 0)
 			(hide yes)
@@
 			)
 		)
-		(property "MPN" "GRM188R72A103KA01D"
+		(property "MPN" "GRM21BR72A103KA01L"
 			(at 190.5 88.9 0)
 			(hide yes)
