File: Power_Indicators.kicad_sch (KiCad schematic)
At the start: 18 parts

Commit message: Add +12V bulk capacitor, document XT30 polarity decision, use E96 values
Input (sheet 1, near J2):
- C36: 220 uF / 35 V low-ESR electrolytic (Panasonic EEU-FR1V221,
  8 x 11.5 mm radial) on +12V right after F1.
- Reverse polarity: no P-FET; rely on the keyed XT30. Note on sheet 1
  and in docs/power-supply.md: the housing cannot mate reversed, but a
  harness crimped backwards at the battery lugs is not caught (it would
  reverse-bias both bucks and C36 until F1 blows), so meter-check harness
  polarity before first power-up and after rework.

All resistor values are now E96:
- R4 40k -> 41.2k 1%: Pi rail 5.12 V (5.1 V target)
- R15 40k -> 40.2k 1%: AUX rail 5.02 V
- R8/R9 31.2k/10k -> 35.7k/11.5k: LDO 3.284 V (31.2k is E192)
- R3 510 -> 511, R21-R24 680 -> 681, R17/R10/R11 4.7k -> 4.75k
Regulator design notes, sheet notes and docs updated to match.
Parts:
- R17: value 4.7k -> 4.75k
- R21, R22, R23, R24: value 680 -> 681
- R3: value 510 -> 511
Other:
- note added: "LED current ~2-2.7 mA: R = (Vrail - 2.0 V) / I. +12V uses 4.75k for the 10.8-14.6 V battery range. All resistors 0805; worst-case dissipation 34 mW (R17 at 14.6 V)."
- note added: "PA5 LED_USER: heartbeat PB12 LED_PI_LINK: Pi UART activity PB13 LED_IMU: IMU data-ready PB14 LED_MOTOR: motor running / fault 681R: (3.3 - 2.1) / 681 = 1.8 mA per pin"
- note removed: "LED current ~2-2.7 mA: R = (Vrail - 2.0 V) / I. +12V uses 4.7k for the 10.8-14.6 V battery range. All resistors 0805; worst-case dissipation 34 mW (R17 at 14.6 V)."
- note removed: "PA5 LED_USER: heartbeat PB12 LED_PI_LINK: Pi UART activity PB13 LED_IMU: IMU data-ready PB14 LED_MOTOR: motor running / fault 680R: (3.3 - 2.1) / 680 = 1.8 mA per pin"
Changed lines of the file:
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@@
 		(company "Senior Design")
 	)
-	(text "LED current ~2-2.7 mA: R = (Vrail - 2.0 V) / I. +12V uses 4.7k for the 10.8-14.6 V battery range.\nAll resistors 0805; worst-case dissipation 34 mW (R17 at 14.6 V)."
+	(text "LED current ~2-2.7 mA: R = (Vrail - 2.0 V) / I. +12V uses 4.75k for the 10.8-14.6 V battery range.\nAll resistors 0805; worst-case dissipation 34 mW (R17 at 14.6 V)."
 		(exclude_from_sim no)
 		(at 50.8 129.54 0)
@@
 		)
 	)
-	(text "PA5 LED_USER: heartbeat\nPB12 LED_PI_LINK: Pi UART activity\nPB13 LED_IMU: IMU data-ready\nPB14 LED_MOTOR: motor running / fault\n680R: (3.3 - 2.1) / 680 = 1.8 mA per pin"
+	(text "PA5 LED_USER: heartbeat\nPB12 LED_PI_LINK: Pi UART activity\nPB13 LED_IMU: IMU data-ready\nPB14 LED_MOTOR: motor running / fault\n681R: (3.3 - 2.1) / 681 = 1.8 mA per pin"
 		(exclude_from_sim no)
 		(at 165.1 116.84 0)
@@
 			)
 		)
-		(property "Value" "510"
+		(property "Value" "511"
 			(at 83.82 116.84 90)
 			(show_name no)
@@
 			)
 		)
-		(property "Value" "680"
+		(property "Value" "681"
 			(at 172.72 66.04 90)
 			(show_name no)
@@
 			)
 		)
-		(property "Description" "Current limit for debug LED D8 on PA5: (3.3 V - 2.1 V) / 680 = 1.8 mA"
+		(property "Description" "Current limit for debug LED D8 on PA5: (3.3 V - 2.1 V) / 681 = 1.8 mA"
 			(at 172.72 63.5 0)
 			(hide yes)
@@
 			)
 		)
-		(property "Value" "680"
+		(property "Value" "681"
 			(at 172.72 91.44 90)
 			(show_name no)
@@
 			)
 		)
-		(property "Description" "Current limit for debug LED D10 on PB13: (3.3 V - 2.1 V) / 680 = 1.8 mA"
+		(property "Description" "Current limit for debug LED D10 on PB13: (3.3 V - 2.1 V) / 681 = 1.8 mA"
 			(at 172.72 88.9 0)
 			(hide yes)
@@
 			)
 		)
-		(property "Value" "680"
+		(property "Value" "681"
 			(at 172.72 78.74 90)
 			(show_name no)
@@
 			)
 		)
-		(property "Description" "Current limit for debug LED D9 on PB12: (3.3 V - 2.1 V) / 680 = 1.8 mA"
+		(property "Description" "Current limit for debug LED D9 on PB12: (3.3 V - 2.1 V) / 681 = 1.8 mA"
 			(at 172.72 76.2 0)
 			(hide yes)
@@
 			)
 		)
-		(property "Value" "680"
+		(property "Value" "681"
 			(at 172.72 104.14 90)
 			(show_name no)
@@
 			)
 		)
-		(property "Description" "Current limit for debug LED D11 on PB14: (3.3 V - 2.1 V) / 680 = 1.8 mA"
+		(property "Description" "Current limit for debug LED D11 on PB14: (3.3 V - 2.1 V) / 681 = 1.8 mA"
 			(at 172.72 101.6 0)
 			(hide yes)
@@
 			)
 		)
-		(property "Value" "4.7k"
+		(property "Value" "4.75k"
 			(at 83.82 66.04 90)
 			(show_name no)
