File: Power_Indicators.kicad_sch (KiCad schematic)
At the start: 18 parts

Commit message: Rename power nets, add mounting holes, retitle sheet 1, clear ERC
Power nets, no commas, named by function:
- "+5V, 2A" -> +5V_SYS, "+5V, 6A PI" -> +5V_PI, "+5V, 6A AUX" -> +5V_AUX
Buck sheets renamed to Buck 5V SYS / Buck 5V PI / Buck 5V AUX. Notes,
descriptions, README and docs updated.

Mechanical and title:
- H1-H4: M3 mounting holes, 3.2 mm plated, isolated (no net), not in BOM
- Sheet 1 title: "Delivery Robot Main Board"

ERC, now 0 errors and 0 warnings (was 4 errors, 15 warnings):
- PWR_FLAGs on +12V (after F1), GND (at J2), +3.3VA (after FB2) and
  +5V_SYS (after the TPS54202's L1)
- TPSM63606 symbol pin types set (VOUT power out, FB/EN input, VIN/
  VLDOIN/GND power in, PG open collector, others passive) in both buck
  sheets and libs/TPSM63606RDLR.kicad_sym
- U1 STM32F091RCTx and Y3 Crystal_GND24 moved to a new
  libs/project_symbols.kicad_sym holding the versions this design uses
  (the current KiCad library moved their pins); libs/TPS54202DDCR made
  to match the schematic's U3
Connectivity unchanged: same 108 nets and pins.

Co-Authored-By: Claude Opus 5.5 <noreply@anthropic.com>
Connections:
- net +5V, 2A renamed +5V_SYS
- net +5V, 6A AUX renamed +5V_AUX
- net +5V, 6A PI renamed +5V_PI
Changed lines of the file:
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@@
 		)
 	)
-	(global_label "+5V, 6A PI"
+	(global_label "+5V_PI"
 		(shape input)
 		(at 76.2 76.2 180)
@@
 		)
 	)
-	(global_label "+5V, 6A AUX"
+	(global_label "+5V_AUX"
 		(shape input)
 		(at 76.2 88.9 180)
@@
 		)
 	)
-	(global_label "+5V, 2A"
+	(global_label "+5V_SYS"
 		(shape input)
 		(at 76.2 101.6 180)
@@
 			)
 		)
-		(property "Description" "Current limit for the +5V, 6A AUX power LED D6: 2.0 mA"
+		(property "Description" "Current limit for the +5V_AUX power LED D6: 2.0 mA"
 			(at 83.82 88.9 0)
 			(hide yes)
@@
 			)
 		)
-		(property "Description" "+5V, 2A rail power indicator, 0603 green LED (2.0 V typ, 571 nm)"
+		(property "Description" "+5V_SYS rail power indicator, 0603 green LED (2.0 V typ, 571 nm)"
 			(at 96.52 101.6 0)
 			(hide yes)
@@
 			)
 		)
-		(property "Description" "+5V, 6A PI rail power indicator, 0603 green LED (2.0 V typ, 571 nm)"
+		(property "Description" "+5V_PI rail power indicator, 0603 green LED (2.0 V typ, 571 nm)"
 			(at 96.52 76.2 0)
 			(hide yes)
@@
 			)
 		)
-		(property "Description" "Current limit for the +5V, 6A PI power LED D5: 2.0 mA"
+		(property "Description" "Current limit for the +5V_PI power LED D5: 2.0 mA"
 			(at 83.82 76.2 0)
 			(hide yes)
@@
 			)
 		)
-		(property "Description" "Current limit for the +5V, 2A power LED D7: 2.0 mA"
+		(property "Description" "Current limit for the +5V_SYS power LED D7: 2.0 mA"
 			(at 83.82 101.6 0)
 			(hide yes)
@@
 			)
 		)
-		(property "Description" "+5V, 6A AUX rail power indicator, 0603 green LED (2.0 V typ, 571 nm)"
+		(property "Description" "+5V_AUX rail power indicator, 0603 green LED (2.0 V typ, 571 nm)"
 			(at 96.52 88.9 0)
 			(hide yes)

Commit message: Remove the IMU from the board; it will be wired off-board
The BNO085 IMU is now connected discretely off the PCB, so everything
for it is removed from the schematic and the layout:
- Delete the IMU Interface sheet (IMU_Interface.kicad_sch): J11 STEMMA
  QT connector, J12 INT/RST header, DNP I2C pull-ups R10/R11 and series
  resistors R34/R35; remove its sheet block, note and project entry
- Remove debug LED D10 / R23 (LED_IMU on PB13)
- Rename the freed MCU nets back to plain pins, still broken out on the
  GPIO headers: IMU_SCL -> PB6, IMU_SDA -> PB7 (J9), IMU_INT -> PC4,
  IMU_RST -> PC5 (J10), LED_IMU -> PB13 (J9)
- Drop IMU wiring notes and the IMU 3.3 V budget line from the LDO sheet;
  update the J9/J10 pin descriptions, debug-LED note and README

Board updated to match (as Update PCB from Schematic): the eight
unplaced footprints deleted, pad nets renamed, J9/J10 descriptions
synced. ERC 0; DRC unchanged at 57 with 276 unrouted (was 293);
schematic parity clean.

Co-Authored-By: Claude Opus 5.5 <noreply@anthropic.com>
Parts:
- removed D10: YELLOW, LED_SMD:LED_0603_1608Metric, symbol Device:LED
- removed R23: 681, Resistor_SMD:R_0805_2012Metric, symbol Device:R
Other:
- note added: "PA5 LED_USER: heartbeat PB12 LED_PI_LINK: Pi UART activity PB14 LED_MOTOR: motor running / fault 681R: (3.3 - 2.1) / 681 = 1.8 mA per pin"
- note removed: "PA5 LED_USER: heartbeat PB12 LED_PI_LINK: Pi UART activity PB13 LED_IMU: IMU data-ready PB14 LED_MOTOR: motor running / fault 681R: (3.3 - 2.1) / 681 = 1.8 mA per pin"
