File: Power_Indicators.kicad_sch (KiCad schematic)
At the start: 16 parts

Commit message: Route the board and apply the prototype PCB checklist fixes
Routing
- Route power (pours, In2 power areas, vias) and all signals; add a
  Signal net class (0.15 mm width/clearance) for low-speed nets.
- J8 expansion header is now a 2x8 near the MCU.

Checklist red flags
- Crystal Y3 moved beside U1's OSC pins with C5/C6 outboard and no
  other signals under it.
- Vias untented by default (tented only under silkscreen); 15 mil
  test vias on key signals, recorded as DRC exclusions.
- ESD: U6/U7 split into four USBLC6-2SC6 (U6, U11, U7, U12), one per
  connector, with VBUS caps C50/C51; R12/R13 moved next to J13.
- GND test loop TP3 moved to the top edge beside J5.

Improvements
- Encoder connectors J7/J15 changed to keyed JST XH S4B side-entry.
- 43 passives/LEDs/FB2 moved from 0603 to 0805 (MPNs updated).
- Fifth M3 mounting hole H5 under J8.
- +3.3VA rerouted away from the crystal; acute track angles removed.
- Datasheet links filled in; silkscreen pin labels, pin maps, team
  names and date; reference labels cleared off pads and vias.
- Custom DRC rule for the J7/J15 silkscreen edge overhang.
Parts:
- D11, D8, D9: footprint LED_SMD:LED_0603_1608Metric -> LED_SMD:LED_0805_2012Metric; MPN LTST-C190KSKT -> LTST-C170KSKT
- D3, D4, D5, D6, D7: footprint LED_SMD:LED_0603_1608Metric -> LED_SMD:LED_0805_2012Metric; MPN LTST-C190KGKT -> LTST-C170KGKT
Changed lines of the file:
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@@
 			)
 		)
-		(property "Footprint" "LED_SMD:LED_0603_1608Metric"
+		(property "Footprint" "LED_SMD:LED_0805_2012Metric"
 			(at 96.52 114.3 0)
 			(hide yes)
@@
 			)
 		)
-		(property "Datasheet" "https://www.futureelectronics.com/p/semiconductors--optoelectronics--leds/ltst-c190kgkt-lite-on-6605018"
+		(property "Datasheet" "https://www.digikey.com/en/products/detail/lite-on-inc/LTST-C170KGKT/386777"
 			(at 96.52 114.3 0)
 			(hide yes)
@@
 			)
 		)
-		(property "MPN" "LTST-C190KGKT"
+		(property "MPN" "LTST-C170KGKT"
 			(at 96.52 114.3 0)
 			(hide yes)
@@
 			)
 		)
-		(property "Footprint" "LED_SMD:LED_0603_1608Metric"
+		(property "Footprint" "LED_SMD:LED_0805_2012Metric"
 			(at 185.42 63.5 0)
 			(hide yes)
@@
 			)
 		)
-		(property "Datasheet" "https://www.lcsc.com/product-detail/Light-Emitting-Diodes-LED_SMD-yellow_C125095.html"
+		(property "Datasheet" "https://datasheet.lcsc.com/lcsc/1810231512_Lite-On-LTST-C170KSKT_C125091.pdf"
 			(at 185.42 63.5 0)
 			(hide yes)
@@
 			)
 		)
-		(property "MPN" "LTST-C190KSKT"
+		(property "MPN" "LTST-C170KSKT"
 			(at 185.42 63.5 0)
 			(hide yes)
@@
 			)
 		)
-		(property "Footprint" "LED_SMD:LED_0603_1608Metric"
+		(property "Footprint" "LED_SMD:LED_0805_2012Metric"
 			(at 185.42 101.6 0)
 			(hide yes)
@@
 			)
 		)
-		(property "Datasheet" "https://www.lcsc.com/product-detail/Light-Emitting-Diodes-LED_SMD-yellow_C125095.html"
+		(property "Datasheet" "https://datasheet.lcsc.com/lcsc/1810231512_Lite-On-LTST-C170KSKT_C125091.pdf"
 			(at 185.42 101.6 0)
 			(hide yes)
@@
 			)
 		)
-		(property "MPN" "LTST-C190KSKT"
+		(property "MPN" "LTST-C170KSKT"
 			(at 185.42 101.6 0)
 			(hide yes)
@@
 			)
 		)
-		(property "Footprint" "LED_SMD:LED_0603_1608Metric"
+		(property "Footprint" "LED_SMD:LED_0805_2012Metric"
 			(at 96.52 101.6 0)
 			(hide yes)
@@
 			)
 		)
-		(property "Datasheet" "https://www.futureelectronics.com/p/semiconductors--optoelectronics--leds/ltst-c190kgkt-lite-on-6605018"
+		(property "Datasheet" "https://www.digikey.com/en/products/detail/lite-on-inc/LTST-C170KGKT/386777"
 			(at 96.52 101.6 0)
 			(hide yes)
@@
 			)
 		)
-		(property "MPN" "LTST-C190KGKT"
+		(property "MPN" "LTST-C170KGKT"
 			(at 96.52 101.6 0)
 			(hide yes)
@@
 			)
 		)
-		(property "Footprint" "LED_SMD:LED_0603_1608Metric"
+		(property "Footprint" "LED_SMD:LED_0805_2012Metric"
 			(at 96.52 76.2 0)
 			(hide yes)
@@
 			)
 		)
-		(property "Datasheet" "https://www.futureelectronics.com/p/semiconductors--optoelectronics--leds/ltst-c190kgkt-lite-on-6605018"
+		(property "Datasheet" "https://www.digikey.com/en/products/detail/lite-on-inc/LTST-C170KGKT/386777"
 			(at 96.52 76.2 0)
 			(hide yes)
@@
 			)
 		)
-		(property "MPN" "LTST-C190KGKT"
+		(property "MPN" "LTST-C170KGKT"
 			(at 96.52 76.2 0)
 			(hide yes)
@@
 			)
 		)
-		(property "Footprint" "LED_SMD:LED_0603_1608Metric"
+		(property "Footprint" "LED_SMD:LED_0805_2012Metric"
 			(at 96.52 63.5 0)
 			(hide yes)
@@
 			)
 		)
-		(property "Datasheet" "https://www.futureelectronics.com/p/semiconductors--optoelectronics--leds/ltst-c190kgkt-lite-on-6605018"
+		(property "Datasheet" "https://www.digikey.com/en/products/detail/lite-on-inc/LTST-C170KGKT/386777"
 			(at 96.52 63.5 0)
 			(hide yes)
@@
 			)
 		)
-		(property "MPN" "LTST-C190KGKT"
+		(property "MPN" "LTST-C170KGKT"
 			(at 96.52 63.5 0)
 			(hide yes)
@@
 			)
 		)
-		(property "Footprint" "LED_SMD:LED_0603_1608Metric"
+		(property "Footprint" "LED_SMD:LED_0805_2012Metric"
 			(at 185.42 76.2 0)
 			(hide yes)
@@
 			)
 		)
-		(property "Datasheet" "https://www.lcsc.com/product-detail/Light-Emitting-Diodes-LED_SMD-yellow_C125095.html"
+		(property "Datasheet" "https://datasheet.lcsc.com/lcsc/1810231512_Lite-On-LTST-C170KSKT_C125091.pdf"
 			(at 185.42 76.2 0)
 			(hide yes)
@@
 			)
 		)
-		(property "MPN" "LTST-C190KSKT"
+		(property "MPN" "LTST-C170KSKT"
 			(at 185.42 76.2 0)
 			(hide yes)
@@
 			)
 		)
-		(property "Footprint" "LED_SMD:LED_0603_1608Metric"
+		(property "Footprint" "LED_SMD:LED_0805_2012Metric"
 			(at 96.52 88.9 0)
 			(hide yes)
@@
 			)
 		)
-		(property "Datasheet" "https://www.futureelectronics.com/p/semiconductors--optoelectronics--leds/ltst-c190kgkt-lite-on-6605018"
+		(property "Datasheet" "https://www.digikey.com/en/products/detail/lite-on-inc/LTST-C170KGKT/386777"
 			(at 96.52 88.9 0)
 			(hide yes)
@@
 			)
 		)
-		(property "MPN" "LTST-C190KGKT"
+		(property "MPN" "LTST-C170KGKT"
 			(at 96.52 88.9 0)
 			(hide yes)
