File: delivery_robot_1.kicad_pcb (KiCad board)
At the start: 4 copper layers, 100 x 100 mm, 114 parts, among them J1 SWD, J10 Port C/D breakout, J11 IMU I2C (STEMMA QT), J12 IMU INT/RST, J13 Pi 5 UART, J14 Pi 5 power, J15 Motor2 encoder, J16 MDD20A PWM2/DIR2/GND, J2 XT30PW-M, J4 BOOT0 jumper, J5 Power test points, J6 MDD20A PWM1/DIR1/GND, J7 Motor1 encoder, J8 Port A breakout, J9 Port B breakout, SW1 RESET, U1 STM32F091RCTx, U2 PTPSM63606RDLR, U3 TPS54202DDCR, U4 TPS7A8101DRBR, U5 PTPSM63606RDLR, U6 USBLC6-4SC6, U7 USBLC6-4SC6, Y3 8MHz

Commit message: Remove the IMU from the board; it will be wired off-board
The BNO085 IMU is now connected discretely off the PCB, so everything
for it is removed from the schematic and the layout:
- Delete the IMU Interface sheet (IMU_Interface.kicad_sch): J11 STEMMA
  QT connector, J12 INT/RST header, DNP I2C pull-ups R10/R11 and series
  resistors R34/R35; remove its sheet block, note and project entry
- Remove debug LED D10 / R23 (LED_IMU on PB13)
- Rename the freed MCU nets back to plain pins, still broken out on the
  GPIO headers: IMU_SCL -> PB6, IMU_SDA -> PB7 (J9), IMU_INT -> PC4,
  IMU_RST -> PC5 (J10), LED_IMU -> PB13 (J9)
- Drop IMU wiring notes and the IMU 3.3 V budget line from the LDO sheet;
  update the J9/J10 pin descriptions, debug-LED note and README

Board updated to match (as Update PCB from Schematic): the eight
unplaced footprints deleted, pad nets renamed, J9/J10 descriptions
synced. ERC 0; DRC unchanged at 57 with 276 unrouted (was 293);
schematic parity clean.

Co-Authored-By: Claude Opus 5.5 <noreply@anthropic.com>
Parts:
- removed D10: YELLOW, LED_SMD:LED_0603_1608Metric
- removed J11: IMU I2C (STEMMA QT), Connector_JST:JST_SH_SM04B-SRSS-TB_1x04-1MP_P1.00mm_Horizontal
- removed J12: IMU INT/RST, Connector_PinHeader_2.54mm:PinHeader_1x02_P2.54mm_Vertical
- removed R10, R11: 4.75k, Resistor_SMD:R_0805_2012Metric
- removed R23: 681, Resistor_SMD:R_0805_2012Metric
- removed R34, R35: 100, Resistor_SMD:R_0805_2012Metric
Connections:
- net IMU_INT renamed PC4
- net IMU_RST renamed PC5
- net IMU_SCL renamed PB6
- net IMU_SDA renamed PB7
- net LED_IMU renamed PB13
