File: delivery_robot_1.kicad_pcb (KiCad board)
At the start: 4 copper layers, 100 x 100 mm, 105 parts, among them J1 SWD, J10 Port C/D breakout, J13 Pi 5 UART, J14 Pi 5 power, J15 Motor2 encoder, J16 MDD20A PWM2/DIR2/GND, J2 XT30PW-M, J4 BOOT0 jumper, J5 Power test points, J6 MDD20A PWM1/DIR1/GND, J7 Motor1 encoder, J8 Port A breakout, J9 Port B breakout, SW1 RESET, U1 STM32F091RCTx, U2 PTPSM63606RDLR, U3 TPS54202DDCR, U4 TPS7A8101DRBR, U5 PTPSM63606RDLR, U6 USBLC6-4SC6, U7 USBLC6-4SC6, Y3 8MHz

Commit message: Place LED and resistor groups, route 3.3 V rails, relabel LEDs
Layout:
- Place D5, TP3, UART series resistors R12/R13 and resistors R3,
  R17-R22, R24 and R26-R33.
- Move C1, and the motor-side regulators U6/U7 with C34/C35.
- Route +3V3, +3.3VA, BOOT and GND tracks; add one copper zone.
- Rename the power/status LED references to rail names
  (D3 -> 3V3, D4 -> 12V, D6 -> AUX, D7 -> SYS, D8 -> HB, D9 -> PI,
  D11 -> MOT). These no longer match the schematic references.
- Unlock the previously locked placements for rework.

Schematic:
- Shorten the J13 note in Pi5_Interface (drop the Pi header pin
  numbers for TXD/RXD).

Co-Authored-By: Claude Opus 5.5 <noreply@anthropic.com>
Parts:
- moved TP2 214.5 mm to (1.68, 1.68)
- moved R26 163.4 mm to (143.7, 132.5), turned to -90 degrees
- moved R27 158.8 mm to (147.3, 132.5), turned to -90 degrees
- moved R30 144.7 mm to (160.6, 136.4), turned to 90 degrees
- moved R31 138.5 mm to (165.5, 135.3), turned to 90 degrees
- moved R32 130.8 mm to (171.4, 132.9)
- moved R28 129.7 mm to (167.5, 109.4)
- moved R29 127.5 mm to (167.5, 105.8)
- moved R33 127.1 mm to (171.4, 127.0)
- moved R20 119.6 mm to (107.8, 58.2), turned to 90 degrees
- moved R3 119.4 mm to (102.5, 58.2), turned to -90 degrees
- moved R19 116.0 mm to (110.6, 58.1), turned to -90 degrees
- moved R18 115.0 mm to (100.0, 90.8), turned to -90 degrees
- moved 3V3 114.2 mm to (102.5, 61.5), turned to 90 degrees
- moved R12 113.9 mm to (164.1, 79.7), turned to -90 degrees
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- renumbered D4 to 12V, D3 to 3V3, D6 to AUX, D8 to HB, D11 to MOT, D9 to PI, D7 to SYS
Routing:
- net +3V3: track 0.00 -> 15.8 mm
- net +3.3VA: track 0.00 -> 5.11 mm
- net BOOT: track 0.00 -> 3.90 mm
- net GND: track 31.5 -> 30.7 mm
- added copper zone on In1.Cu, net GND
