File: Pi5_Interface.kicad_sch (KiCad schematic)
At the start: 7 parts, among them J13 Pi 5 UART, J14 Pi 5 power

Commit message: Place buck converters, connectors and Pi power path on the PCB
Layout:
- Place the U2 (+5V_PI) 6 A buck group, and a copy of the same layout
  for the U5 (+5V_AUX) buck: U5, C28-C33, R14-R16.
- Place the U3 2 A buck (L1, R6/R7, C14-C17), the remaining J
  connectors (J1, J4, J5, J8-J10, J13, J14) and test point TP1.
- Add copper zones and vias. Set the default zone pad connection to
  solid.

Schematic:
- Remove F2 from the Pi 5 power path; +5V_PI now feeds J14 directly.
Parts:
- removed F2: 7.5A / 32VDC, Fuse:Fuseholder_Blade_Mini_Keystone_3568, symbol Device:Fuse
Connections:
- net VIN_5V: now also J14.1 (Pin_1), TP2.1
Changed lines of the file:
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@@
 	(wire
 		(pts
-			(xy 69.85 124.46) (xy 77.47 124.46)
+			(xy 69.85 124.46) (xy 92.71 124.46)
 		)
 		(stroke
@@
 		(pts
 			(xy 97.79 127) (xy 97.79 129.54)
-		)
-		(stroke
-			(width 0)
-			(type default)
-		)
-	)
-	(wire
-		(pts
-			(xy 85.09 124.46) (xy 92.71 124.46)
 		)
 		(stroke
@@
 		)
 	)
-	(symbol
-		(lib_id "Device:Fuse")
-		(at 81.28 124.46 270)
-		(unit 1)
-		(body_style 1)
-		(exclude_from_sim no)
-		(in_bom yes)
-		(on_board yes)
-		(in_pos_files yes)
-		(dnp no)
-		(fields_autoplaced yes)
-		(property "Reference" "F2"
-			(at 81.28 118.11 90)
-			(show_name no)
-			(do_not_autoplace no)
-			(effects
-				(font
-					(size 1.27 1.27)
-				)
-			)
-		)
-		(property "Value" "7.5A / 32VDC"
-			(at 81.28 120.65 90)
-			(show_name no)
-			(do_not_autoplace no)
-			(effects
-				(font
-					(size 1.27 1.27)
-				)
-			)
-		)
-		(property "Footprint" "Fuse:Fuseholder_Blade_Mini_Keystone_3568"
-			(at 81.28 122.68 90)
-			(hide yes)
-			(show_name no)
-			(do_not_autoplace no)
-			(effects
-				(font
-					(size 1.27 1.27)
-				)
-			)
-		)
-		(property "Datasheet" "https://www.keyelco.com/product-pdf.cfm?p=306"
-			(at 81.28 124.46 0)
-			(hide yes)
-			(show_name no)
-			(do_not_autoplace no)
-			(effects
-				(font
-					(size 1.27 1.27)
-				)
-			)
-		)
-		(property "Description" "Pi 5 supply isolation and fuse: Keystone 3568 holder and Littelfuse 029707.5L 7.5 A fuse. Remove the fuse to isolate the Pi for buck bring-up; 6.0 A allowed at 40 C per Littelfuse derating table, above the Pi 5 5 A maximum."
-			(at 81.28 124.46 0)
-			(hide yes)
-			(show_name no)
-			(do_not_autoplace no)
-			(effects
-				(font
-					(size 1.27 1.27)
-				)
-			)
-		)
-		(property "Manufacturer" "Keystone Electronics"
-			(at 81.28 124.46 0)
-			(hide yes)
-			(show_name no)
-			(do_not_autoplace no)
-			(effects
-				(font
-					(size 1.27 1.27)
-				)
-			)
-		)
-		(property "MPN" "3568"
-			(at 81.28 124.46 0)
-			(hide yes)
-			(show_name no)
-			(do_not_autoplace no)
-			(effects
-				(font
-					(size 1.27 1.27)
-				)
-			)
-		)
-		(property "Specification" "MINI holder with 7.5A / 32VDC fuse; 1000A DC interrupt rating belongs to fuse"
-			(at 81.28 124.46 0)
-			(hide yes)
-			(show_name no)
-			(do_not_autoplace no)
-			(effects
-				(font
-					(size 1.27 1.27)
-				)
-			)
-		)
-		(property "FuseManufacturer" "Littelfuse"
-			(at 81.28 124.46 0)
-			(hide yes)
-			(show_name no)
-			(do_not_autoplace no)
-			(effects
-				(font
-					(size 1.27 1.27)
-				)
-			)
-		)
-		(property "FuseMPN" "029707.5L"
-			(at 81.28 124.46 0)
-			(hide yes)
-			(show_name no)
-			(do_not_autoplace no)
-			(effects
-				(font
-					(size 1.27 1.27)
-				)
-			)
-		)
-		(property "FuseDatasheet" "https://www.littelfuse.com/assetdocs/littelfuse-datasheet-297-mini32v?assetguid=42c9dd21-a88e-4328-8e67-2f832444faf1"
-			(at 81.28 124.46 0)
-			(hide yes)
-			(show_name no)
-			(do_not_autoplace no)
-			(effects
-				(font
-					(size 1.27 1.27)
-				)
-			)
-		)
-		(property "AssemblyBOM" "1x Keystone 3568 holder + 1x Littelfuse 029707.5L fuse; order both"
-			(at 81.28 124.46 0)
-			(hide yes)
-			(show_name no)
-			(do_not_autoplace no)
-			(effects
-				(font
-					(size 1.27 1.27)
-				)
-			)
-		)
-		(pin "2"
-		)
-		(pin "1"
-		)
-		(instances
-			(project "delivery_robot_1"
-				(path "/30314d9c-15a8-4a77-8ae4-b5ba12ed5bc4/c056b61f-6369-4e88-a9e3-647282746e13"
-					(reference "F2")
-					(unit 1)
-				)
-			)
-		)
-	)
