File: Pi5_Interface.kicad_sch (KiCad schematic)
At the start: 11 parts, among them J13 Pi 5 link, J14 Pi 5 power, Q2 DMN63D8L

Commit message: Switch AUX ports to top-entry JST XH; drop encoder pull-ups and Pi sense
- J18-J21 (peripheral 5 V ports) are now top-entry JST XH B2B-XH-A:
  cables plug in from above, which suits a flat board you reach into,
  and the footprint drops from 107 to 58 mm2 per port. Use pre-made
  2-pin XH cables, so no crimping.
- Remove the DNP encoder pull-ups R48-R51. If the am-3651 outputs turn
  out to be open-collector, bodge 4.7k from each A/B line to ENCn_5V
  (noted on the Motor Control sheet).
- Remove the Pi-alive sense R44/R45. PA1 is a spare pin again (J8 pin
  2); the Pi's 3V3 on J13 still enables the AUX buck through D15.
- Board: same edits as Update PCB from Schematic (J18-J21 swapped,
  six resistors deleted, PA1 net restored on U1/J8); the parked parts
  are re-grouped beside the board. Venya's tracks unchanged (87).
- Docs, README and schematic PDF updated.

ERC 0/0. DRC: 0 errors, 3 existing text-size warnings, parity clean.
Parts:
- removed R44: 10k, Resistor_SMD:R_0805_2012Metric, symbol Device:R
- removed R45: 100k, Resistor_SMD:R_0805_2012Metric, symbol Device:R
Other:
- note added: "Pi-controlled functions (J13 4 <- Pi 3V3 pin 1, 5 <- GPIO23 pin 16, 6 <- GPIO24 pin 18) AUX_EN: the +5V_AUX buck (U5) runs only while the Pi's 3V3 is up. PI_RESET + PI_BOOT0 -> reflash the STM32 from the Pi over USART2 (AN2606: PA2/PA3 is a bootloader port on STM32F09x). Sequence: BOOT0 high, pulse reset, run stm32flash at 115200 8E1, then BOOT0 low and reset. At Pi boot GPIO23/24 default to pull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"
- note removed: "Pi-controlled functions (J13 4 <- Pi 3V3 pin 1, 5 <- GPIO23 pin 16, 6 <- GPIO24 pin 18) AUX_EN: the +5V_AUX buck (U5) runs only while the Pi's 3V3 is up. PI_3V3_SENSE -> PA1: firmware can tell whether the Pi is alive. PI_RESET + PI_BOOT0 -> reflash the STM32 from the Pi over USART2 (AN2606: PA2/PA3 is a bootloader port on STM32F09x). Sequence: BOOT0 high, pulse reset, run stm32flash at 115200 8E1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"
