File: Buck_5V_2A.kicad_sch (KiCad schematic)
At the start: 8 parts, among them U3 TPS54202DDCR

Commit message: Add motor 1 driver and encoder screw terminals
Label the STM32 pins used in the motor prototype: PA6 MOTOR1_PWM
(TIM3_CH1 to DRI0002 E1), PB0 MOTOR1_DIR (M1), PA15 ENC1_A and PB3
ENC1_B (TIM2 encoder inputs).

Add screw terminals to the right of U1:
- J6, 3-pos: MOTOR1_PWM, MOTOR1_DIR, GND for the DFRobot DRI0002
- J7, 4-pos: +5V 2A, ENC1_A, ENC1_B, GND for the 37D motor encoder
Encoder power comes from the +5V 2A buck rail ahead of the LDO.

Both use Phoenix MKDS 1,5 5.0 mm footprints (1715035, 1715048),
rated 17.5 A / 250 V for the 5 V, 2 A requirement, with datasheet,
part number and pinout stored in the symbol properties.

Also includes the sheet layout rearranged in KiCad.

Co-Authored-By: Claude Opus 5.5 <noreply@anthropic.com>
Other:
- note added: "12 V - 5 V, 2A Buck Convertor"
- note added: "Reusable sheet: VIN_12V input, VOUT_5V output, common GND"
- note removed: "Reusable sheet: VIN_12V input, VOUT_5V output, common GND VOUT set by R6/R7 divider on FB; fixed 500 kHz; L1 15 uH; C15 is the BOOT-SW bootstrap cap. EN is flagged no-connect - confirm floating EN is allowed in the datasheet."
- moved on the sheet: C14, C15, C16, C17, L1, R6, R7, U3

Commit message: Rename power nets, add mounting holes, retitle sheet 1, clear ERC
Power nets, no commas, named by function:
- "+5V, 2A" -> +5V_SYS, "+5V, 6A PI" -> +5V_PI, "+5V, 6A AUX" -> +5V_AUX
Buck sheets renamed to Buck 5V SYS / Buck 5V PI / Buck 5V AUX. Notes,
descriptions, README and docs updated.

Mechanical and title:
- H1-H4: M3 mounting holes, 3.2 mm plated, isolated (no net), not in BOM
- Sheet 1 title: "Delivery Robot Main Board"

ERC, now 0 errors and 0 warnings (was 4 errors, 15 warnings):
- PWR_FLAGs on +12V (after F1), GND (at J2), +3.3VA (after FB2) and
  +5V_SYS (after the TPS54202's L1)
- TPSM63606 symbol pin types set (VOUT power out, FB/EN input, VIN/
  VLDOIN/GND power in, PG open collector, others passive) in both buck
  sheets and libs/TPSM63606RDLR.kicad_sym
- U1 STM32F091RCTx and Y3 Crystal_GND24 moved to a new
  libs/project_symbols.kicad_sym holding the versions this design uses
  (the current KiCad library moved their pins); libs/TPS54202DDCR made
  to match the schematic's U3
Connectivity unchanged: same 108 nets and pins.

Co-Authored-By: Claude Opus 5.5 <noreply@anthropic.com>
Parts:
- U3: Used In Sheet Buck_5V_2A: 12 V in, +5V 2A net out (feeds LDO sheet) -> Sheet Buck_5V_2A: 12 V in, +5V_SYS net out (feeds LDO sheet)
Changed lines of the file:
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@@
 			)
 		)
-		(property "Used In" "Sheet Buck_5V_2A: 12 V in, +5V 2A net out (feeds LDO sheet)"
+		(property "Used In" "Sheet Buck_5V_2A: 12 V in, +5V_SYS net out (feeds LDO sheet)"
 			(at 135.89 90.17 0)
 			(hide yes)

Commit message: Add input protection, AUX ports, servo interface and Pi control
Implements the 2026-10-15 design review decisions in the schematic.
ERC 0 errors, 0 warnings.

New sheets:
- Input Protection: Q1 SQJ409EP reverse-battery P-FET after F1 (D12
  12 V gate clamp, R36), D13 SMBJ16A TVS on +12V, battery sense
  R37/R38/C37 -> VBAT_SENSE on PA0. PWR_FLAG moves to +12V.
- AUX Outputs: four +5V_AUX ports J18-J21 (JST XH 2-pin: Notecard,
  LiDAR, GNSS, IMU), each through a 1.5 A PTC (F4-F7).
- Servo Interface: J17 (GND, VBAT_SERVO via F3 5 A fuse, SERVO_SIG) for
  the Hiwonder HTS-30HS through an external 11.1-12 V buck. U8
  SN74LVC1T45 translates PB10 (USART3 half-duplex) to the 5 V bus,
  PB11 sets direction; R39-R42 pull-ups/series, D14 ESD.

Root sheet:
- F1 output is now VBAT_FUSED; C36 sits on +12V after Q1. J2-F1 net
  named VBAT_IN. F1 7.5 A -> 10 A (0297010.L).
- Y3/C5/C6 fitted (were DNP).
- PA0 -> VBAT_SENSE, PA1 -> PI_3V3_SENSE, PB10 -> SERVO_TX,
  PB11 -> SERVO_DIR. Notes updated (no more F2 / XT30-only text).

Pi 5 Interface:
- J13 -> 6-pin JST XH: TXD, RXD, GND, PI_3V3, PI_RESET, PI_BOOT0.
- PI_3V3 -> D15 -> AUX_EN (U5 enable) and R44/R45 -> PA1.
- PI_RESET -> Q2 DMN63D8L -> NRST (open drain, R46 pull-down).
- PI_BOOT0 -> R47 1k -> BOOT0, for reflashing over USART2.
- R12/R13 100R -> 1k (PA2/PA3 are TTa, 5 mA injection max).
- Remove TP2 (same net as TP1 since F2 was removed).

Buck 5V AUX: U5 EN from AUX_EN (was +12V), R43 100k pull-down, C40,
J22 force-on jumper. Buck 5V SYS: C49 100 nF at U3 VIN/GND.
U2/U5 value TPSM63606RDLR; VCC design note corrected (internal 1 uF,
must stay NC).

Motor Control (now A3):
- U9/U10 74LVC2G17 encoder buffers on +3V3; encoder series R 100R ->
  1k with C43-C46 1 nF; R48-R51 4.7k pull-ups (DNP).
- F8/F9 0.2 A PTC + C47/C48 on each encoder supply (ENC1_5V, ENC2_5V).
- J7/J15 pin order 5V, GND, A, B (matches the am-3651 plug).
- R52/R53 10k pull-downs on both PWM lines (MDD20A brakes on low).
- F10/F11 PTC in series with J6/J16 p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
Parts:
- added C49: 100nF / 50V X7R, Capacitor_SMD:C_0603_1608Metric, symbol Device:C
Connections:
- net GND: now also C49.2
- net VIN_12V: now also C49.1
Changed lines of the file:
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@@
+	)
+	(junction
+		(at 111.76 107.95)
+		(diameter 0)
+		(color 0 0 0 0)
 	)
 	(junction
 		(at 167.64 81.28)
+		(diameter 0)
+		(color 0 0 0 0)
+	)
+	(junction
+		(at 111.76 82.55)
 		(diameter 0)
 		(color 0 0 0 0)
@@
 	(wire
 		(pts
+			(xy 111.76 82.55) (xy 111.76 85.09)
+		)
+		(stroke
+			(width 0)
+			(type default)
+		)
+	)
+	(wire
+		(pts
 			(xy 156.21 82.55) (xy 153.67 82.55)
 		)
@@
 		(pts
 			(xy 106.68 82.55) (xy 106.68 85.09)
+		)
+		(stroke
+			(width 0)
+			(type default)
+		)
+	)
+	(wire
+		(pts
+			(xy 111.76 92.71) (xy 111.76 107.95)
 		)
 		(stroke
@@
 		)
 	)
+	(symbol
+		(lib_id "Device:C")
+		(at 111.76 88.9 0)
+		(unit 1)
+		(body_style 1)
+		(exclude_from_sim no)
+		(in_bom yes)
+		(on_board yes)
+		(in_pos_files yes)
+		(dnp no)
+		(property "Reference" "C49"
+			(at 114.3 87.63 0)
+			(show_name no)
+			(do_not_autoplace no)
+			(effects
+				(font
+					(size 1.27 1.27)
+				)
+				(justify left)
+			)
+		)
+		(property "Value" "100nF / 50V X7R"
+			(at 114.3 90.17 0)
+			(show_name no)
+			(do_not_autoplace no)
+			(effects
+				(font
+					(size 1.27 1.27)
+				)
+				(justify left)
+			)
+		)
+		(property "Footprint" "Capacitor_SMD:C_0603_1608Metric"
+			(at 111.76 88.9 0)
+			(hide yes)
+			(show_name no)
+			(do_not_autoplace no)
+			(effects
+				(font
+					(size 1.27 1.27)
+				)
+			)
+		)
+		(property "Datasheet" "~"
+			(at 111.76 88.9 0)
+			(hide yes)
+			(show_name no)
+			(do_not_autoplace no)
+			(effects
+				(font
+					(size 1.27 1.27)
+				)
+			)
+		)
+		(property "Description" "High-frequency input cap for U3, right at VIN (pin 3) and GND (pin 1). C14 (2220) is the bulk part; this small one keeps the switching loop short (TI SLVSD26C 7.2.3.1 and 7.4.1)."
+			(at 111.76 88.9 0)
+			(hide yes)
+			(show_name no)
+			(do_not_autoplace no)
+			(effects
+				(font
+					(size 1.27 1.27)
+				)
+			)
+		)
+		(property "Manufacturer" "KEMET"
+			(at 111.76 88.9 0)
+			(hide yes)
+			(show_name no)
+			(do_not_autoplace no)
+			(effects
+				(font
+					(size 1.27 1.27)
+				)
+			)
+		)
+		(property "MPN" "C0603C104K5RACTU"
+			(at 111.76 88.9 0)
+			(hide yes)
+			(show_name no)
+			(do_not_autoplace no)
+			(effects
+				(font
+					(size 1.27 1.27)
+				)
+			)
+		)
+		(pin "1"
+		)
+		(pin "2"
+		)
+		(instances
+			(project "delivery_robot_1"
+				(path "/30314d9c-15a8-4a77-8ae4-b5ba12ed5bc4/45fd30b8-e3d0-4ad8-a19a-9569735f4754"
+					(reference "C49")
+					(unit 1)
+				)
+			)
+		)
+	)
