File: Motor_Control.kicad_sch (KiCad schematic)
At the start: 16 parts, among them J15 Motor2 encoder, J16 MDD20A PWM2/DIR2/GND, J6 MDD20A PWM1/DIR1/GND, J7 Motor1 encoder, U6 USBLC6-4SC6, U7 USBLC6-4SC6

Commit message: Rename power nets, add mounting holes, retitle sheet 1, clear ERC
Power nets, no commas, named by function:
- "+5V, 2A" -> +5V_SYS, "+5V, 6A PI" -> +5V_PI, "+5V, 6A AUX" -> +5V_AUX
Buck sheets renamed to Buck 5V SYS / Buck 5V PI / Buck 5V AUX. Notes,
descriptions, README and docs updated.

Mechanical and title:
- H1-H4: M3 mounting holes, 3.2 mm plated, isolated (no net), not in BOM
- Sheet 1 title: "Delivery Robot Main Board"

ERC, now 0 errors and 0 warnings (was 4 errors, 15 warnings):
- PWR_FLAGs on +12V (after F1), GND (at J2), +3.3VA (after FB2) and
  +5V_SYS (after the TPS54202's L1)
- TPSM63606 symbol pin types set (VOUT power out, FB/EN input, VIN/
  VLDOIN/GND power in, PG open collector, others passive) in both buck
  sheets and libs/TPSM63606RDLR.kicad_sym
- U1 STM32F091RCTx and Y3 Crystal_GND24 moved to a new
  libs/project_symbols.kicad_sym holding the versions this design uses
  (the current KiCad library moved their pins); libs/TPS54202DDCR made
  to match the schematic's U3
Connectivity unchanged: same 108 nets and pins.

Co-Authored-By: Claude Opus 5.5 <noreply@anthropic.com>
Connections:
- net +5V, 2A renamed +5V_SYS

Commit message: Add input protection, AUX ports, servo interface and Pi control
Implements the 2026-10-15 design review decisions in the schematic.
ERC 0 errors, 0 warnings.

New sheets:
- Input Protection: Q1 SQJ409EP reverse-battery P-FET after F1 (D12
  12 V gate clamp, R36), D13 SMBJ16A TVS on +12V, battery sense
  R37/R38/C37 -> VBAT_SENSE on PA0. PWR_FLAG moves to +12V.
- AUX Outputs: four +5V_AUX ports J18-J21 (JST XH 2-pin: Notecard,
  LiDAR, GNSS, IMU), each through a 1.5 A PTC (F4-F7).
- Servo Interface: J17 (GND, VBAT_SERVO via F3 5 A fuse, SERVO_SIG) for
  the Hiwonder HTS-30HS through an external 11.1-12 V buck. U8
  SN74LVC1T45 translates PB10 (USART3 half-duplex) to the 5 V bus,
  PB11 sets direction; R39-R42 pull-ups/series, D14 ESD.

Root sheet:
- F1 output is now VBAT_FUSED; C36 sits on +12V after Q1. J2-F1 net
  named VBAT_IN. F1 7.5 A -> 10 A (0297010.L).
- Y3/C5/C6 fitted (were DNP).
- PA0 -> VBAT_SENSE, PA1 -> PI_3V3_SENSE, PB10 -> SERVO_TX,
  PB11 -> SERVO_DIR. Notes updated (no more F2 / XT30-only text).

Pi 5 Interface:
- J13 -> 6-pin JST XH: TXD, RXD, GND, PI_3V3, PI_RESET, PI_BOOT0.
- PI_3V3 -> D15 -> AUX_EN (U5 enable) and R44/R45 -> PA1.
- PI_RESET -> Q2 DMN63D8L -> NRST (open drain, R46 pull-down).
- PI_BOOT0 -> R47 1k -> BOOT0, for reflashing over USART2.
- R12/R13 100R -> 1k (PA2/PA3 are TTa, 5 mA injection max).
- Remove TP2 (same net as TP1 since F2 was removed).

Buck 5V AUX: U5 EN from AUX_EN (was +12V), R43 100k pull-down, C40,
J22 force-on jumper. Buck 5V SYS: C49 100 nF at U3 VIN/GND.
U2/U5 value TPSM63606RDLR; VCC design note corrected (internal 1 uF,
must stay NC).

Motor Control (now A3):
- U9/U10 74LVC2G17 encoder buffers on +3V3; encoder series R 100R ->
  1k with C43-C46 1 nF; R48-R51 4.7k pull-ups (DNP).
- F8/F9 0.2 A PTC + C47/C48 on each encoder supply (ENC1_5V, ENC2_5V).
- J7/J15 pin order 5V, GND, A, B (matches the am-3651 plug).
- R52/R53 10k pull-downs on both PWM lines (MDD20A brakes on low).
- F10/F11 PTC in series with J6/J16 p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
Parts:
- added C41, C42: 100nF / 50V X7R, Capacitor_SMD:C_0603_1608Metric, symbol Device:C
- added C43, C44, C45, C46: 1nF / 50V C0G, Capacitor_SMD:C_0603_1608Metric, symbol Device:C
- added C47, C48: 1uF / 16V X7R, Capacitor_SMD:C_0603_1608Metric, symbol Device:C
- added F10, F11, F8, F9: 0.2A hold, Fuse:Fuse_1206_3216Metric, symbol Device:Polyfuse
- added R48, R49, R50, R51: 4.7k, Resistor_SMD:R_0805_2012Metric, symbol Device:R
- added R52, R53: 10k, Resistor_SMD:R_0805_2012Metric, symbol Device:R
- added U10, U9: 74LVC2G17, Package_TO_SOT_SMD:SOT-23-6, symbol 74xGxx:74LVC2G17
- R28, R29, R32, R33: value 100 -> 1k
Connections:
- net +3V3: now also C41.1, C42.1, U10.5 (VCC), U9.5 (VCC)
- net +5V_SYS: now also F8.1, F9.1; no longer J15.1 (Pin_1), J7.1 (Pin_1)
- net ENC1_A: now also U9.6; no longer R28.1
- net ENC1_A_CONN: now also J7.3 (Pin_3), R48.2; no longer J7.2 (Pin_2)
- net ENC1_B: now also U9.4; no longer R29.1
- net ENC1_B_CONN: now also J7.4 (Pin_4), R49.2; no longer J7.3 (Pin_3)
- net ENC2_A: now also U10.6; no longer R32.1
- net ENC2_A_CONN: now also J15.3 (Pin_3), U7.4 (I/O3), R50.2; no longer J15.2 (Pin_2)
- net ENC2_B: now also U10.4; no longer R33.1
- net ENC2_B_CONN: now also J15.4 (Pin_4), U7.6 (I/O4), R51.2; no longer J15.3 (Pin_3)
- net GND: now also J15.2 (Pin_2), J7.2 (Pin_2), C41.2, C42.2, C43.2, C44.2, C45.2, C46.2, C47.2, C48.2, F10.2, F11.2, R52.2, R53.2, U10.2 (GND), U9.2 (GND); no longer J15.4 (Pin_4), J16.3 (Pin_3), J6.3 (Pin_3), J7.4 (Pin_4)
- net MOTOR1_PWM_CONN: now also R52.1
- net MOTOR2_DIR_CONN: now also U6.6 (I/O4)
- net MOTOR2_PWM_CONN: now also U6.4 (I/O3), R53.1
- new net ENC1_5V: C47.1, F8.2, J7.1 (Pin_1), R48.1, R49.1
- new net ENC1_A_F: C43.1, R28.1, U9.1
- new net ENC1_B_F: C44.1, R29.1, U9.3
- new net ENC2_5V: C48.1, F9.2, J15.1 (Pin_1), R50.1, R51.1
- new net ENC2_A_F: C45.1, R32.1, U10.1
- new net ENC2_B_F: C46.1, R33.1, U10.3
- new net M1_DRV_GND: F10.1, J6.3 (Pin_3)
- new net M2_DRV_GND: F11.1, J16.3 (Pin_3)
- no-connect marks 4 -> 0
Other:
- note added: "ESD arrays - U6: J6 + J16, U7: J7 + J15"
- note added: "Encoder input buffers - 74LVC2G17 on +3V3 (inputs tolerate 5.5 V, even unpowered)"
- note added: "Encoder supply, encoder pull-ups (DNP), motor-driver line protection"
- note added: "Motor control - Cytron MDD20A dual-channel driver + two AndyMark PG27 motors with am-3651 encoders"
- note added: "STM32F091 PIN ASSIGNMENT series R connector MOTOR1_PWM PA6 TIM3_CH1 R26 100R J6 pin 1 -> MDD20A PWM1 (R52 10k pull-down) MOTOR1_DIR PB0 GPIO R27 100R J6 pin 2 -> MDD20A DIR1 ENC1_A PA15 TIM2_CH1 U9 <- R28 1k J7 pin 3 <- encoder A ENC1_B PB3 TIM2_CH2 U9 <- R29 1k J7 pin 4 <- encoder B MOTOR2_PWM PA7 TIM3_CH2 R30 100R J16 pin 1 -> MDD20A PWM2 (R53 10k pull-down) MOTOR2_DIR PB2 GPIO R31 100R J16 pin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"
- note added: "Series resistors (MCU side): 100R driver lines, 1k encoder lines"
- note removed: "ESD arrays - J6 and J7 only"
- note removed: "Motor control - Cytron MDD20A dual-channel driver + two 37D encoder motors"
- note removed: "STM32F091 PIN ASSIGNMENT series R connector MOTOR1_PWM PA6 TIM3_CH1 R26 100R J6 pin 1 -> MDD20A PWM1 MOTOR1_DIR PB0 GPIO R27 100R J6 pin 2 -> MDD20A DIR1 ENC1_A PA15 TIM2_CH1 R28 100R J7 pin 2 <- encoder A (yellow) ENC1_B PB3 TIM2_CH2 R29 100R J7 pin 3 <- encoder B (white) MOTOR2_PWM PA7 TIM3_CH2 R30 100R J16 pin 1 -> MDD20A PWM2 MOTOR2_DIR PB2 GPIO R31 100R J16 pin 2 -> MDD20A DIR2 ENC2_A PA8 TI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"
- note removed: "Series 100R (MCU side)"
