File: Servo_Interface.kicad_sch (KiCad schematic)
At the start: 10 parts, among them J17 Latch servo, U8 SN74LVC1T45DBV

Commit message: Route the board and apply the prototype PCB checklist fixes
Routing
- Route power (pours, In2 power areas, vias) and all signals; add a
  Signal net class (0.15 mm width/clearance) for low-speed nets.
- J8 expansion header is now a 2x8 near the MCU.

Checklist red flags
- Crystal Y3 moved beside U1's OSC pins with C5/C6 outboard and no
  other signals under it.
- Vias untented by default (tented only under silkscreen); 15 mil
  test vias on key signals, recorded as DRC exclusions.
- ESD: U6/U7 split into four USBLC6-2SC6 (U6, U11, U7, U12), one per
  connector, with VBUS caps C50/C51; R12/R13 moved next to J13.
- GND test loop TP3 moved to the top edge beside J5.

Improvements
- Encoder connectors J7/J15 changed to keyed JST XH S4B side-entry.
- 43 passives/LEDs/FB2 moved from 0603 to 0805 (MPNs updated).
- Fifth M3 mounting hole H5 under J8.
- +3.3VA rerouted away from the crystal; acute track angles removed.
- Datasheet links filled in; silkscreen pin labels, pin maps, team
  names and date; reference labels cleared off pads and vias.
- Custom DRC rule for the J7/J15 silkscreen edge overhang.
Parts:
- C38, C39: footprint Capacitor_SMD:C_0603_1608Metric -> Capacitor_SMD:C_0805_2012Metric; MPN C0603C104K5RACTU -> C0805C104K5RACTU
Changed lines of the file:
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@@
 			)
 		)
-		(property "Footprint" "Capacitor_SMD:C_0603_1608Metric"
+		(property "Footprint" "Capacitor_SMD:C_0805_2012Metric"
 			(at 106.68 87.63 0)
 			(hide yes)
@@
 			)
 		)
-		(property "Datasheet" "~"
+		(property "Datasheet" "https://content.kemet.com/datasheets/KEM_C1002_X7R_SMD.pdf"
 			(at 106.68 87.63 0)
 			(hide yes)
@@
 			)
 		)
-		(property "MPN" "C0603C104K5RACTU"
+		(property "MPN" "C0805C104K5RACTU"
 			(at 106.68 87.63 0)
 			(hide yes)
@@
 			)
 		)
-		(property "Datasheet" ""
+		(property "Datasheet" "https://www.phoenixcontact.com/en-us/products/pcb-terminal-block-mkds-15-3-1715035"
 			(at 213.36 76.2 0)
 			(hide yes)
@@
 			)
 		)
-		(property "Footprint" "Capacitor_SMD:C_0603_1608Metric"
+		(property "Footprint" "Capacitor_SMD:C_0805_2012Metric"
 			(at 127 87.63 0)
 			(hide yes)
@@
 			)
 		)
-		(property "Datasheet" "~"
+		(property "Datasheet" "https://content.kemet.com/datasheets/KEM_C1002_X7R_SMD.pdf"
 			(at 127 87.63 0)
 			(hide yes)
@@
 			)
 		)
-		(property "MPN" "C0603C104K5RACTU"
+		(property "MPN" "C0805C104K5RACTU"
 			(at 127 87.63 0)
 			(hide yes)
